Commit message: forgot some files

File: parol6/urdf_model/urdf/PAROL6.urdf (robot description, URDF)
Before this commit: robot parol6, 9 links, 8 joints
Links:
- removed link tool0
Joints:
- removed joint L6_to_tool0

Commit message: added tools

File: parol6/urdf_model/urdf/PAROL6.urdf (robot description, URDF)
Before this commit: robot parol6, 8 links, 7 joints
Joints:
- joint L6: origin xyz=0 0.0628 0 rpy=1.5707963267949 0 0 -> xyz=0 0.044 0 rpy=1.5707963267949 0 0

Commit message: add tcp_offset commands and fix planner tool sync on RESET
- new SET_TCP_OFFSET / TCP_OFFSET wire commands; SetTcpOffsetCommand
  is a SystemCommand and now lives in SYSTEM_CMD_TYPES so the client
  waits for ack instead of leaving stale OK in the rx queue
- TCP_OFFSET added to QUERY_CMD_TYPES for consistency
- controller now syncs tool state to the planner subprocess on RESET
  (fixes test_cartesian_move_validation when run after tool tests)
- joint_path_to_tcp_poses uses pinokin so3_rpy (intrinsic XYZ) to
  match the convention used elsewhere in robot.py
- async_client move_s/move_p Category: Smooth Motion -> Motion to
  match the ABC; drop incompatible move_j @overloads
- examples reorganised to mirror programs/ (deleted pick_and_place,
  reachable poses in demo_showcase, use robot.create_sync_client)
- example tests gated behind --examples flag (port 5001 collides
  with the integration server fixture); 240s subprocess + 300s
  pytest timeout per example

File: parol6/urdf_model/urdf/PAROL6.urdf (robot description, URDF)
Before this commit: robot parol6, 8 links, 7 joints
Joints:
- joint L6: origin xyz=0 0.044 0 rpy=1.5707963267949 0 0 -> xyz=0 0.037 0 rpy=1.5707963267949 0 0
